File: pcb/kowgary16_cfx/kowgary16_cfx.kicad_pcb (KiCad board)
At the start: 2 copper layers, 170 x 69.4 mm, 104 parts, among them J1 USB_C_Receptacle_USB2.0, SW1 SW_Push, SW10 SW_Push, SW11 SW_Push, SW12 SW_Push, SW13 SW_Push, SW14 SW_Push, SW15 SW_Push, SW16 SW_Push, SW17 SW_Push, SW18 SW_Push, SW19 SW_Push, SW2 SW_Push, SW20 SW_Push, SW21 SW_Push, SW22 SW_Push, SW23 SW_Push, SW24 SW_Push, SW25 SW_Push, SW26 SW_Push, SW27 SW_Push, SW28 SW_Push, SW29 SW_Push, SW3 SW_Push, SW30 SW_Push, SW31 SW_Push, SW32 SW_Push, SW33 SW_Push, SW34 SW_Push, SW35 SW_Push, SW36 SW_Push, SW37 SW_Push, SW38 SW_Push, SW39 SW_Push, SW4 SW_Push, SW40 SW_Push, SW5 SW_Push, SW6 SW_Push, SW7 SW_Push, SW8 SW_Push, SW9 SW_Push, U1 ATmega32U4-M, Y1 16MHz

Commit message: init commit
Parts:
- removed D10, D15, D16, D17, D18, D19, D20, D25, D26, D27, D28, D29, D30, D35, D36, D37, D38, D39, D40, D5, D6, D7, D8, D9: D_Small, Diode_SMD:D_SOD-323
- removed H5, H6: MountingHole, MountingHole:MountingHole_2.2mm_M2_ISO7380
- removed SW10, SW15, SW16, SW17, SW18, SW19, SW20, SW25, SW26, SW27, SW28, SW29, SW30, SW35, SW36, SW37, SW38, SW39, SW40, SW5, SW6, SW7, SW8, SW9: SW_Push, keyswitches:Kailh_socket_PG1350
- H1, H2, H3, H4: moved to B.Cu
- R4, R5: value 22 -> 22R
- moved H4 103.4 mm to (125.4, 65.9), turned to 180 degrees
- moved H2 102.0 mm to (91.4, 31.9), turned to 180 degrees
- moved H3 17.0 mm to (91.4, 65.9), turned to 180 degrees
- turned H1 to 180 degrees
Connections:
- U1 pad 18: col10 -> unconnected-(U1-Pad18)
- U1 pad 19: col9 -> unconnected-(U1-Pad19)
- U1 pad 20: col8 -> unconnected-(U1-Pad20)
- U1 pad 21: col7 -> unconnected-(U1-Pad21)
- U1 pad 22: col6 -> unconnected-(U1-Pad22)
- U1 pad 25: col5 -> unconnected-(U1-Pad25)
Routing:
- net col7: track 201.3 -> 0.00 mm, vias 3 -> 0
- net col10: track 176.9 -> 0.00 mm, vias 2 -> 0
- net col9: track 173.0 -> 0.00 mm, vias 2 -> 0
- net col8: track 146.0 -> 0.00 mm, vias 2 -> 0
- net col6: track 126.0 -> 0.00 mm, vias 2 -> 0
- net row2: track 223.5 -> 109.5 mm, vias 16 -> 10
- net row1: track 192.2 -> 78.3 mm, vias 16 -> 7
- net row3: track 210.7 -> 97.0 mm, vias 17 -> 11
- net row4: track 228.4 -> 115.2 mm, vias 15 -> 9
- net col5: track 102.7 -> 0.00 mm, vias 2 -> 0
- net GND: track 121.0 -> 133.7 mm
- net col1: track 77.2 -> 80.4 mm
- net col2: track 74.4 -> 77.3 mm, vias 2 -> 4
- net Net-(D8-Pad2): track 2.42 -> 0.00 mm
- net Net-(D5-Pad2): track 2.42 -> 0.00 mm
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Other:
- board size 170 x 69.4 mm -> 68 x 69.4 mm
- board text added: "kowgary16 by sporewoh v0.0"
- board text added: "イーホー!!"
- board text removed: "bancouver40 by sporewoh v0.0"
- board text removed: "please work please work please work"
